File: Hardware/8ModuleBoard/8ModuleBoard.sch (EAGLE design)
At the start: 18 parts, among them X1 MKS1854-6-0-404

Commit message: Updated the Hardware and software drives
Parts:
- added ATMEGA32U4: ATMEGA32U4TQFP-44, SparkFun-DigitalIC:ATMEGA32U4TQFP-44
- added B1, B2, B3: DBDB101G, rectifier:DBDB101G
- added BLE: BLE_Extn, con-molex:22-23-2051
- added C10, C18, C19, C6: 0.1uF, SparkFun-Passives:CAP1206
- added C11, C12, C13: 2.2uF/63V, rcl:CPOL-EUE1.8-4
- added C14, C16: 2.2uF/250VAC, capacitor-wima:C27/9
- added C15, C17: 3.3uF/250VAC, capacitor-wima:C27/9
- added C7: 1uF, SparkFun-Passives:CAP1206
- added C8, C9: 18pF, SparkFun-Passives:CAP1206
- added CN1: com-BUS, con-molex:22-23-2081
- added CN2: Capsense I/P, con-molex:22-23-2081
- added CX1, CX2, CX3: 220nF/275V~, rcl:CXXC15B5
- added D2, D4, D6: 1N4007, gm-diodes:1N400X.1
- added D3, D5, D7: 10V/0W4, diode:ZENER-DIODEZD-2.5
- added H1, H2, H3, H4, H5, H6, H7, H8: MOUNT-HOLE2.8, holes:MOUNT-HOLE2.8
- added IR: IR_CON, con-molex:22-23-2031
- added IR1, IR2: PNA460XM, adafruit:PNA460XM
- added JP2: USB-Programming, SparkFun-Connectors:USB-MICROB
- added JP3: USB-Charging, SparkFun-Connectors:USB-A-H
- added KK1, KK2, KK3: SK95-2M3, heatsink:SK95-2M3
- added LED3: (no value), led:LEDSML1206
- added LED6, LED7: (no value), led:LEDSMT1206
- added LOAD_CN: (no value), con-ptr500:AK300/8
- added OK1, OK2, OK3: 4N35, optocoupler:4N35
- added OK4, OK5, OK6, OK7, OK8: MOC3031M, optocoupler:MOC3031M
- added PWR, X3, X5: 22-23-2031, con-molex:22-23-2031
- added Q1: 16MHz, crystal:CRYSTALHC49UP
- added Q2, Q3, Q4: IRF840, transistor-fet:IRF840
- added R12, R13, R22: 220R, SparkFun-Resistors:RESISTOR1206
- added R14, R15, R18, R19, R23, R24: 33K/1W, rcl:R-EU_0411/3V
- added R16, R20, R25, R9: 1K, SparkFun-Passives:RESISTOR1206
- added R17, R21, R26: 22K, SparkFun-Passives:RESISTOR1206
- added R27, R29, R31, R33, R35: 560R, SparkFun-Resistors:RESISTOR1206
- added R28, R30, R32, R34, R36: 470R/0.5W, rcl:R-US_0411/3V
- added R37: 39R/2W, rcl:R-EU_0411/3V
- added R38, R41: 470R, SparkFun-Passives:RESISTOR1206
- added R39, R40, R42, R43: 1K, SparkFun-Resistors:RESISTOR1206
- added R6: 10K, SparkFun-Passives:RESISTOR1206
- added R7, R8: 22R, SparkFun-Passives:RESISTOR1206
- added RN1: (no value), resistor-sil:G07R
- added SMPS_5V@2A: 5V@2A, Morsun-con-stocko:MKS1854-6-0-404
- added T1, T2, T3, T4, T5: BTB16-V, triac:BT138-V
- added U$11, U$3: HM-11, HM-11:HM-11
- added U$4, U$6, U$8: 220K, SparkFun-Resistors:RESISTOR1206
- added U$5, U$7, U$9: 2E2, SparkFun-Resistors:RESISTOR1206
- added X4: 22-23-2051, con-molex:22-23-2051
- C1: value (none) -> 470uF/25V
- C2: value (none) -> 0.01uF/400V; device rcl:CPOL-EUE5-8.5 -> capacitor-wima:C2.5/2
- C3: value 1.0uF -> 0.1uF
- F1: value (none) -> PFUSE 1A
- LED1, LED2: device led:LEDSMT1206 -> led:LEDSML1206
- R1: value S05K300 -> MOV300V; device varistor:S05K300 -> varistor:S07K11
- R2: value (none) -> 1K
- R3: value (none) -> 470R
- R4, R5: value (none) -> 1K; device SparkFun-Passives:RESISTOR1206 -> SparkFun-Resistors:RESISTOR1206
- X1: value MKS1854-6-0-404 -> 22-23-2051; device Morsun-con-stocko:MKS1854-6-0-404 -> con-molex:22-23-2051
- renumbered X2 to AC
Connections:
- removed net N$8: U$1.UART_CTS
- new net !RESET: ATMEGA32U4.!RESET, BLE-5.S, CN1-4.S, R6.1, U$3.UART_RTS
- new net BGND: IR1.GND, LED6.C, U$1.GND, X1-2.S, X3-2.S
- new net BLE_STATUS: R3.2, U$3.PIO1
- new net CGND: IR2.GND, LED7.C, U$11.GND, X4-2.S, X5-2.S
- new net DIMM1: ATMEGA32U4.PB6(ADC13), R16.1
- new net DIMM2: ATMEGA32U4.PC6, R20.1
- new net DIMM3: ATMEGA32U4.PC7, R25.1, R9.2
- new net DOWN: ATMEGA32U4.PB4(ADC11), CN2-7.S, RN1.7
- new net FAN_ON/OFF: ATMEGA32U4.PB5(ADC12), CN2-8.S, RN1.8
- new net FAN_REG: LOAD_CN-8.KL, T4.A1, U$5.1, U$7.1, U$9.1
- new net IR_RX: ATMEGA32U4.PB7, IR-1.S
- new net LEVEL1: ATMEGA32U4.PF6(ADC6), R27.1
- new net LEVEL2: ATMEGA32U4.PF5(ADC5), R29.1
- new net LEVEL3: ATMEGA32U4.PF4(ADC4), R31.1
- new net LEVEL4: ATMEGA32U4.PF1(ADC1), R33.1
- new net LINE: B1.AC2, B2.AC2, B3.AC2, F1.2, LOAD_CN-1.KL, R1.2, R28.2, R30.2, R32.2, R34.2, R36.2, R37.2, SMPS_5V@2A.L, T1.A2, T2.A2, T3.A2, T4.A2, T5.A2
- new net LOAD_1: B1.AC1, LOAD_CN-4.KL
- new net LOAD_2: B2.AC1, LOAD_CN-5.KL
- new net LOAD_3: B3.AC1, LOAD_CN-6.KL
- new net MISO: ATMEGA32U4.PB3(MISO), CN1-3.S
- new net N$1: OK6.A, R31.2
- new net N$10: ATMEGA32U4.AREF, C6.1
- new net N$11: R5.2, U$3.UART_RX
- new net N$13: B1.-, C11.-, CX1.2, D3.A, Q2.S, R17.2
- new net N$16: JP2.D-, R7.2
- new net N$17: JP2.D+, R8.2
- new net N$18: ATMEGA32U4.D-, R7.1
- new net N$19: ATMEGA32U4.D+, R8.1
- new net N$20: CX1.1, R13.2, R14.1
- new net N$21: R14.2, R15.1
- new net N$22: ATMEGA32U4.XTAL2, C8.2, Q1.2
- new net N$23: ATMEGA32U4.XTAL1, C9.2, Q1.1
- new net N$24: OK1.A, R16.2
- new net N$25: C11.+, D3.C, OK1.COL, R15.2
- new net N$26: R38.2, U$1.PIO1
- new net N$27: C2.1, R37.1
- new net N$28: OK1.EMI, Q2.G, R17.1
- new net N$29: D4.C, R12.1
- new net N$30: CX2.1, R12.2, R18.1
- new net N$31: ATMEGA32U4.PE6
- new net N$32: B1.+, D2.A, Q2.D
- new net N$33: R18.2, R19.1
- new net N$34: C12.+, D5.C, OK2.COL, R19.2
- new net N$35: OK2.A, R20.2
- new net N$37: OK2.EMI, Q3.G, R21.1
- new net N$38: B2.+, D4.A, Q3.D
- new net N$39: LED6.A, R38.1
- new net N$40: U$1.UART_RTS, X1-5.S
- new net N$41: B3.-, C13.-, CX3.2, D7.A, Q4.S, R26.2
- new net N$42: D6.C, R22.1
- new net N$43: CX3.1, R22.2, R23.1
- new net N$44: ATMEGA32U4.PF7(ADC7)
- new net N$45: R23.2, R24.1
- new net N$46: C13.+, D7.C, OK3.COL, R24.2
- new net N$47: OK3.A, R25.2
- new net N$48: R40.1, X1-4.S
- new net N$49: OK3.EMI, Q4.G, R26.1
- new net N$50: B3.+, D6.A, Q4.D
- new net N$51: R39.1, X1-3.S
- new net N$52: OK4.A2, R28.1
- new net N$54: OK4.A1, T1.G
- new net N$55: C14.1, T1.A1, U$4.2
- new net N$56: C14.2, U$4.1, U$5.2
- new net N$57: U$1.VCC, X1-1.S
- new net N$60: OK5.A2, R30.1
- new net N$61: IR1.OUT, X3-1.S
- new net N$62: OK5.A1, T2.G
- new net N$63: C15.1, T2.A1, U$6.2
- new net N$64: C15.2, U$6.1, U$7.2
- new net N$67: IR1.VCC, X3-3.S
- new net N$68: OK6.A2, R32.1
- new net N$7: ATMEGA32U4.UCAP, C7.2
- new net N$70: OK6.A1, T3.G
- new net N$71: C16.1, C17.1, T3.A1, U$8.2
- new net N$72: C16.2, C17.2, U$8.1, U$9.2
- new net N$76: OK7.A2, R34.1
- new net N$78: OK7.A1, T4.G
- new net N$82: OK8.A2, R36.1
- new net N$84: OK8.A1, T5.G
- new net N$85: R42.2, U$11.UART_TX
- new net N$86: R43.2, U$11.UART_RX
- new net N$87: R41.2, U$11.PIO1
- new net N$88: LED7.A, R41.1
- new net N$89: U$11.UART_RTS, X4-5.S
- new net N$90: R43.1, X4-4.S
- new net N$91: R42.1, X4-3.S
- new net N$93: U$11.VCC, X4-1.S
- new net N$94: IR2.OUT, X5-1.S
- new net N$96: IR2.VCC, X5-3.S
- new net NEUTRAL: AC-2.KL, LOAD_CN-2.KL, LOAD_CN-3.KL, R1.1, SMPS_5V@2A.N
- new net PLUG_CONTROL: C2.2, LOAD_CN-7.KL, T5.A1
- new net R27: OK8.A, R27.2
- new net R29: OK7.A, R29.2
- new net R33: OK5.A, R33.2
- new net R35: OK4.A, R35.2
- new net RX: ATMEGA32U4.PD3(TX), BLE-4.S, R5.1
- new net RX_LED: ATMEGA32U4.PB0(SS)
- new net SCL: ATMEGA32U4.PD0(SCL), CN1-5.S
- new net SDA: ATMEGA32U4.PD1(SDA), CN1-6.S
- new net SOCKET: ATMEGA32U4.PF0(ADC0), R35.1
- new net SW-1: ATMEGA32U4.PB1(SCK), CN1-8.S, CN2-2.S, RN1.2
- new net SW-2: ATMEGA32U4.PB2(MOSI), CN1-7.S, CN2-3.S, RN1.3
- new net SW-3: ATMEGA32U4.PD4(ADC8), CN2-4.S, RN1.4
- new net SW-4: ATMEGA32U4.PD6(ADC9), CN2-5.S, RN1.5
- new net TX: ATMEGA32U4.PD2(RX), BLE-3.S, R4.1
- new net TX_LED: ATMEGA32U4.PD5
- new net UP: ATMEGA32U4.PD7(ADC10), CN2-6.S, RN1.6
- net +3V3: now also BLE-1.S, U$3.VCC
- net +5V: now also ATMEGA32U4.AVCC@24, ATMEGA32U4.AVCC@44, ATMEGA32U4.UVCC, ATMEGA32U4.VBUS, ATMEGA32U4.VCC@14, ATMEGA32U4.VCC@34, C10.2, C18.1, C19.2, CN1-1.S, IR-3.S, JP2.VBUS, JP3.VBUS, PWR-1.S, R6.2, RN1.1, SMPS_5V@2A.V+; no longer C2.+, X1.V+
- net GND: now also ATMEGA32U4.GND@15, ATMEGA32U4.GND@23, ATMEGA32U4.GND@35, ATMEGA32U4.GND@43, ATMEGA32U4.PE2/!HWB, ATMEGA32U4.UGND, BLE-2.S, C10.1, C18.2, C19.1, C6.2, C7.1, C8.1, C9.1, CN1-2.S, CN2-1.S, IR-2.S, JP2.GND, JP3.GND, LED3.C, OK1.C, OK2.C, OK3.C, OK4.C, OK5.C, OK6.C, OK7.C, OK8.C, PWR-2.S, SMPS_5V@2A.GND, U$3.GND; no longer C2.-, X1.GND
- net N$12: now also R40.2, U$1.UART_RX; no longer R5.1
- net N$14: now also D2.C, R13.1; no longer LED2.A, R5.2
- net N$2: now also B2.-, C12.-, CX2.2, D5.A, Q3.S, R21.2; no longer AC-2.KL, R1.1, X1.N
- net N$3: now also R39.2, U$1.UART_TX; no longer F1.2, R1.2, X1.L
- net N$4: now also R4.2, U$3.UART_TX; no longer U$1.UART_RTS
- net N$5: now also LED3.A, R9.1; no longer R3.2, U$1.UART_TX
- net N$9: now also LED2.A, R3.1; no longer R4.2, U$1.UART_RX
Other:
- note added: "Bluetooth Extention"
- note added: "Bluetooth Section"
- note added: "Fan Regulator"
- note added: "LEVEL1"
- note added: "LEVEL2"
- note added: "LEVEL3"
- note added: "LEVEL4"
- note added: "Level-1"
- note added: "Level-2"
- note added: "Level-3"
- note added: "Level-4"
- note added: "Light Dimmer"
- note added: "Microcontroller Unit"
- note added: "Power Supply Section"
- note added: "SOCKET"
- note added: "Socket Control"
- note removed: "BLE Section"
- note removed: "Power Supply Secion"
- moved on the sheet: LED2, R3, R4, R5
