File: Hardware/4Key1SliderCapsenseDesign/4key1SliderCapsenseDesign.brd (EAGLE design)
At the start: 160 x 100 mm, 76 parts, among them T1 BC847, U1 CY8C42XX-44, X1 SWD Interface, X2 22-23-2121, Y1 32.768KHz

Commit message: Updated the Hardware Files with Vr2
Parts:
- added BAT1: (no value), SparkFun-Electromechanical:BATTCON_245MM
- added D7: BAS40-05, diode:SOT23
- added H1, H2, H3, H4: MOUNT-HOLE2.8, holes:2,8
- added L1, L2, L3, L4, L5: (no value), led:CHIPLED_1206
- D2, D3, D4, D5, D6: device SparkFun-LED:LED-1206-BOTTOM -> led:CHIP-LED0805
- moved R28 295.6 mm to (-129.7, 127.8)
- moved R29 294.0 mm to (-128.8, 122.5)
- moved R31 291.2 mm to (96.2, 65.3), flipped to the bottom
- moved R30 289.0 mm to (96.1, 67.8), flipped to the bottom
- moved SW2 271.8 mm to (50.0, 56.0), turned to 90 degrees
- moved SW1 258.9 mm to (25.0, 56.0), turned to 90 degrees
- moved SL2 252.3 mm to (83.3, 66.1)
- moved SW3 251.7 mm to (37.5, 36.5), turned to 90 degrees
- moved SW5 246.8 mm to (50.0, 15.0), turned to 90 degrees
- moved C10 240.7 mm to (-90.7, 117.1)
- moved C12 240.7 mm to (-90.7, 106.9)
- moved C9 240.7 mm to (-90.7, 122.1)
- moved C11 240.7 mm to (-90.7, 112.0)
- moved C13 240.7 mm to (-90.7, 101.8)
- moved SW4 229.9 mm to (25.0, 15.0), turned to 90 degrees
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Connections:
- new net +5V: D7.1, X2.4
- new net N$39: BAT1.1, D7.2
- net GND: now also BAT1.2
- net N$34: now also L1.A, L2.A, L3.A, L4.A, L5.A
- net N$36: now also L1.C, L2.C, L3.C, L4.C, L5.C
- net N$51: now also IR1.VS; no longer IR1.VO
- net VCC: now also D7.3, IR1.VO; no longer IR1.VS, X2.4
Other:
- board size 160 x 100 mm -> 145.3 x 90.2 mm
- board text added: "4- Module Box"
- board text added: "Decop Cap"
- board text added: "Guard Sensor"
- board text added: "RTC"
- board text added: "cutting Area"
- board text added: "proximity Sensor resion"
