File: Hardware/4Key1SliderCapsenseDesign/4key1SliderCapsenseDesign.sch (EAGLE design)
At the start: 76 parts, among them T1 BC847, U1 CY8C42XX-44, X1 SWD Interface, X2 22-23-2121, Y1 32.768KHz

Commit message: Updated the Hardware Files with Vr2
Parts:
- added BAT1: (no value), SparkFun-Electromechanical:BATTERY245MM
- added D7: BAS40-05, diode:BAS40-05
- added H1, H2, H3, H4: MOUNT-HOLE2.8, holes:MOUNT-HOLE2.8
- added L1, L2, L3, L4, L5: (no value), led:LEDCHIPLED_1206
- D2, D3, D4, D5, D6: device SparkFun-LED:LED1206-BOTTOM -> led:LEDCHIP-LED0805
Connections:
- new net +5V: D7.A1, X2-4.S
- new net N$39: BAT1.+, D7.A2
- net GND: now also BAT1.-
- net N$34: now also L1.A, L2.A, L3.A, L4.A, L5.A
- net N$36: now also L1.C, L2.C, L3.C, L4.C, L5.C
- net N$51: now also IR1.VS; no longer IR1.VO
- net VCC: now also D7.C, IR1.VO; no longer IR1.VS, X2-4.S
Other:
- note added: "RTC Battery"
- note added: "To PSoC device"
- note added: "to pin 35"
- note added: "to pin 36"
- note removed: "Add RGB POWER LED for BACK LIGHTING"
