File: Hardware/8ModuleBoard_vr2/8ModuleBoard_vr2.brd (EAGLE design)
At the start: 160 x 100 mm, 78 parts, among them CN2 Capsense I/P, Q1 16MHz, T1 BTB16-V, T2 BTB16-V, T3 BTB16-V, T4 BTB16-V, T5 BTB16-V, U1 LM-35, Y1 32.768KHz

Commit message: Updated with Vr2 of Switchboard
Parts:
- removed C10, C11: 0.1uF, SparkFun-Passives:1206
- removed C2: 0.01uF/400V, capacitor-wima:C2.5-2
- removed JP3: USB-Charging, SparkFun-Connectors:USB-A-H
- removed R35: 560R, SparkFun-Resistors:1206
- removed R36: 470R/0.5W, rcl:0411V
- removed R37: 39R/2W, rcl:0411V
- removed T5: BTB16-V, triac:TO220BV
- removed U$10: RF-LINK_TX, SparkFun-RF:RF-LINK_TX
- removed U1: LM-35, microbuilder:BREAKOUT_SOIC8
- added ANT1: (no value), discrete:PAD-01
- added D10, D11, D4, D5, D6, D7, D8, D9: (no value), diode:SOD123
- added IC2: HT680D, holtek:SOP18
- added JP1: AVR_SPI_PRG_6PTH, SparkFun-Connectors:2X3
- added K1, K2, K3, K4: JS-M1-9V-4, relay:JS-M
- added LED3: (no value), led:SML1206
- added OK1, OK2, OK3: PC817DIL4, optocoupler:DIL4-SMD
- added Q2, Q3, Q4, Q5, Q6: MMBT2222A, SparkFun-DiscreteSemi:SOT23-3
- added R10, R11, R12, R13: S10K11, varistor:S10K11
- added R14: 10K, SparkFun-Passives:1206
- added R15: 560R, SparkFun-Resistors:1206
- added R16: 33k, SparkFun-Resistors:1206
- added R17, R18, R19, R20: 1K, SparkFun-Resistors:1206
- added S1: SWS008, smd-special:SMS-008
- added X1: 22-23-2031, con-molex:22-23-2031
- OK4, OK5, OK6, OK7: value MOC3031M -> MOC3031S; device optocoupler:DIL06 -> optocoupler:DIL6-SMD
- OK8: value MOC3031M -> PC817DIL4; device optocoupler:DIL06 -> optocoupler:DIL4-SMD
- R1: device varistor:S07K11 -> varistor:S10K11
- moved R8 306.4 mm to (113.0, 11.4), flipped to the bottom, turned to 90 degrees
- moved R7 300.9 mm to (110.5, 11.4), flipped to the bottom, turned to 90 degrees
- moved U$2 286.1 mm to (64.4, 3.25)
- moved U$9 278.0 mm to (156.3, 49.2), flipped to the bottom
- moved U$8 257.9 mm to (125.6, 47.4), flipped to the bottom, turned to 180 degrees
- moved U$4 250.9 mm to (156.3, 46.1), flipped to the bottom, turned to 180 degrees
- moved H3 250.3 mm to (177.2, 52.6)
- moved U$6 248.2 mm to (156.3, 52.4), flipped to the bottom, turned to 180 degrees
- moved T1 248.2 mm to (165.6, 1.40), turned to 180 degrees
- moved C15 246.4 mm to (154.3, 53.0), turned to 180 degrees
- moved U$5 245.0 mm to (156.3, 42.8), flipped to the bottom
- moved B1 244.7 mm to (44.6, 30.3)
- moved R33 241.0 mm to (141.5, 36.6), turned to 90 degrees
- moved C14 240.9 mm to (157.9, 45.7), turned to 180 degrees
- moved T2 240.1 mm to (161.3, 12.9), turned to 90 degrees
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Connections:
- removed net N$17: U1.2
- removed net N$18: U1.3
- removed net N$21: R8.2, U$1.5
- removed net N$25: U1.5
- removed net N$26: U1.6
- removed net N$28: U1.7
- removed net N$4 (its old number): OK8.1, R35.2
- removed net N$82: OK8.6, R36.1
- removed net N$84: OK8.4, T5.G
- removed net SOCKET: R35.1
- removed net V_TEMP: U1.1
- new net (DIN)TE: IC2.14, U$2.DATA@1
- new net (VT)ADOUT: IC2.17, R14.2
- new net A0: IC2.1, S1.16
- new net A1: IC2.2, S1.15
- new net A2: IC2.3, S1.14
- new net A3: IC2.4, S1.13
- new net A4: IC2.5, S1.12
- new net A5: IC2.6, S1.11
- new net A6: IC2.7, S1.10
- new net A7: IC2.8, S1.9
- new net D10: ATMEGA32U4.40, IC2.12
- new net D11: ATMEGA32U4.41, IC2.13
- new net D8: ATMEGA32U4.38, IC2.10
- new net D9: ATMEGA32U4.39, IC2.11
- new net MISO: ATMEGA32U4.11, JP1.3, R20.1
- new net MOSI: ATMEGA32U4.10, JP1.5, R19.1
- new net N$24: Q2.3, R15.1
- new net N$31: ANT1.1, U$2.ANT
- new net N$32: OK1.3, Q3.1
- new net N$33: D5.A, K1.2, OK1.4, Q3.3
- new net N$37: D4.C, D5.C
- new net N$38: K1.NC
- new net N$41: OK1.1, R17.2
- new net N$43: OK2.3, Q4.1
- new net N$45: D7.A, K2.2, OK2.4, Q4.3
- new net N$46: D6.C, D7.C
- new net N$47: K2.NC
- new net N$50: OK2.1, R18.2
- new net N$51: OK3.3, Q5.1
- new net N$53: D9.A, K3.2, OK3.4, Q5.3
- new net N$57: D8.C, D9.C
- new net N$58: K3.NC
- new net N$65: OK3.1, R19.2
- new net N$66: OK8.3, Q6.1
- new net N$67: D11.A, K4.2, OK8.4, Q6.3
- new net N$69: D10.C, D11.C
- new net N$73: K4.NC
- new net N$77: OK8.1, R20.2
- new net N$8: Q2.1, R14.1
- new net N$83: ATMEGA32U4.8, R17.1
- new net OSC1: IC2.16, R16.1
- new net OSC2: IC2.15, R16.2
- new net SCK: ATMEGA32U4.9, JP1.4, R18.1
- new net SCL: ATMEGA32U4.18, R7.2, U$1.6
- new net SDA: ATMEGA32U4.19, R8.2, U$1.5
- net !RESET: now also JP1.1
- net +5V: now also D10.A, D4.A, D6.A, D8.A, IC2.18, JP1.2, K1.1, K2.1, K3.1, K4.1, LED3.A, X1.1; no longer C10.2, C11.1, JP3.VBUS, U$10.VCC, U1.8
- net DOWN: now also ATMEGA32U4.29
- net FAN_ON/OFF: now also ATMEGA32U4.30
- net FAN_REG: now also R10.1, R11.1, R12.1, R13.1
- net GND: now also IC2.9, JP1.6, OK1.2, OK2.2, OK3.2, Q2.2, Q3.2, Q4.2, Q5.2, Q6.2, S1.1, S1.2, S1.3, S1.4, S1.5, S1.6, S1.7, S1.8, X1.2; no longer C10.1, C11.2, JP3.GND, U$10.GND, U1.4
- net LEVEL1: now also ATMEGA32U4.31
- net LEVEL2: now also ATMEGA32U4.32
- net LEVEL3: now also ATMEGA32U4.36
- net LEVEL4: now also ATMEGA32U4.37
- net LINE: now also F1.1, K1.C, K2.C, K3.C, K4.C, R10.2, R11.2, R12.2, R13.2; no longer F1.2, R36.2, R37.2, T5.T2
- net LOAD_1: now also K4.NO
- net LOAD_2: now also K1.NO
- net LOAD_3: now also K2.NO
- net N$12: now also Y1.1; no longer Y1.2
- net N$13: now also Y1.2; no longer Y1.1
- net N$20: now also ATMEGA32U4.1; no longer R7.2, U$1.6
- net N$27: now also LED3.C, R15.2; no longer C2.1, R37.1
- net N$36: now also F1.2; no longer F1.1
- net PLUG_CONTROL: now also K3.NO; no longer C2.2, T5.T1
- net RX: now also ATMEGA32U4.21
- net SW-1: now also ATMEGA32U4.22
- net SW-2: now also ATMEGA32U4.25
- net SW-3: now also ATMEGA32U4.26
- net SW-4: now also ATMEGA32U4.27
- net TX: now also ATMEGA32U4.20
- net UP: now also ATMEGA32U4.28
Routing:
- net GND: track 0.00 -> 527.5 mm, vias 0 -> 8
- net N$25: track 0.00 -> 485.9 mm
- net N$21: track 0.00 -> 485.9 mm
- net LINE: track 0.00 -> 402.9 mm
- net +5V: track 0.00 -> 375.8 mm, vias 0 -> 4
- net TX: track 0.00 -> 170.5 mm, vias 0 -> 2
- net FAN_REG: track 0.00 -> 169.9 mm
- net RX: track 0.00 -> 153.2 mm, vias 0 -> 2
- net !RESET: track 0.00 -> 145.8 mm, vias 0 -> 4
- net (DIN)TE: track 0.00 -> 114.4 mm
- net MOSI: track 0.00 -> 83.4 mm, vias 0 -> 3
- net N$14: track 0.00 -> 78.5 mm, vias 0 -> 2
- net N$71: track 0.00 -> 78.1 mm
- net N$55: track 0.00 -> 69.8 mm
- net NEUTRAL: track 0.00 -> 68.8 mm
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- added copper zone on layer 1, net GND
- added copper zone on layer 16, net GND
Other:
- board size 160 x 100 mm -> 181 x 56.6 mm
- board text added: "3.3V Battery"
- board text added: "BOT SIDE"
- board text added: "HBT Vr2"
- board text added: "ICSP"
- board text added: "Made In India"
- board text added: "TOP SIDE"

Commit message: Updated with 8 Module Relay Board Design
Parts:
- added 0, 1, 2, 3, 4, 5, 6, 7, 8, 9, DOWN, F_OFF, F_ON, UP: BUTTON-CONDUCTIVESMD, SparkFun-Electromechanical:BUTTON-CONDUCTIVE
- added ANT2: (no value), discrete:PAD-01
- added D12, D13, D14, D15, D16, D17, D18, D19, D20, D21, D22, D23, D24, D25, D26, D27, D28, D29, D30, D31, D32, D33, D34, D35, D36, D37, D38, D39, D40, D41, D42, D43: (no value), diode:SOD123
- added IC3: HT680D, holtek:SOP18
- added MASTER: BUTTON-CONDUCTIVE, SparkFun-Electromechanical:BUTTON-CONDUCTIVE-MINI
- added R21, R22, R23, R9: 1K, SparkFun-Passives:1206
- added R24: 750K, SparkFun-Passives:1206
- added S2: (no value), SparkFun-Electromechanical:SWITCH-SPST-SMD-A
- added S3: 219-08J, switch-dil:CTS-219-08J
- added TX: RF-LINK_TX, SparkFun-RF:RF-LINK_TX
- added U$10, U$13: (no value), logo:CE-4MM
- added U$11: (no value), logo:FCC_6.1X15MM
- added U$12: (no value), logo:FCC_20X8.35MM
- added VBAT: (no value), SparkFun-Electromechanical:BATTCON_20MM
- moved H4 0.35 mm to (177.0, 3.85)
- moved H1 0.28 mm to (3.83, 52.6)
- moved H3 0.22 mm to (176.9, 52.6)
Connections:
- new net EA0: IC3.1, S3.16
- new net EA1: IC3.2, S3.15
- new net EA2: IC3.3, S3.14
- new net EA3: IC3.4, S3.13
- new net EA4: IC3.5, S3.12
- new net EA5: IC3.6, S3.11
- new net EA6: IC3.7, S3.10
- new net EA7: IC3.8, S3.9
- new net EAD10: D16.C, D18.C, D20.C, D23.C, D34.C, D36.C, D39.C, D42.C, IC3.12, R22.1
- new net EAD11: D24.C, D26.C, D28.C, D31.C, D35.C, D37.C, D40.C, D43.C, IC3.13, R23.1
- new net EAD8: D12.C, D14.C, D17.C, D21.C, D25.C, D29.C, D32.C, D38.C, IC3.10, R9.1
- new net EAD9: IC3.11, R21.1
- new net EDOUT: IC3.17, TX.DATA
- new net EOSC1: IC3.16, R24.2
- new net EOSC2: IC3.15, R24.1
- new net GNDA: IC3.14, IC3.9, R21.2, R22.2, R23.2, R9.2, S3.1, S3.2, S3.3, S3.4, S3.5, S3.6, S3.7, S3.8, TX.GND, VBAT.2
- new net N$17: 1.2, D12.A
- new net N$18: 2.2, D13.A
- new net N$26: S2.2, VBAT.1
- new net N$28: S2.3, TX.VCC
- new net N$35: 3.2, D14.A, D15.A
- new net N$40: ANT2.1, TX.ANT
- new net N$42: 4.2, D16.A
- new net N$44: 5.2, D17.A, D18.A
- new net N$48: 6.2, D19.A, D20.A
- new net N$49: 7.2, D21.A, D22.A, D23.A
- new net N$52: 0.2, D27.A, D28.A
- new net N$59: D13.C, D15.C, D19.C, D22.C, D27.C, D30.C, D33.C, D41.C
- new net N$60: D29.A, D30.A, D31.A, UP.2
- new net N$61: 8.2, D24.A
- new net N$68: D36.A, D37.A, F_ON.2
- new net N$74: 9.2, D25.A, D26.A
- new net N$75: D38.A, D39.A, D40.A, DOWN.2
- new net N$76: D32.A, D33.A, D34.A, D35.A, MASTER.2
- new net N$79: D41.A, D42.A, D43.A, F_OFF.2
- new net V+: 0.1, 1.1, 2.1, 3.1, 4.1, 5.1, 6.1, 7.1, 8.1, 9.1, DOWN.1, F_OFF.1, F_ON.1, IC3.18, MASTER.1, UP.1
Routing:
- net N$80: track 0.00 -> 252.8 mm
- net N$39: track 0.00 -> 252.5 mm
- net EAD11: track 0.00 -> 238.9 mm, vias 0 -> 7
- net V+: track 0.00 -> 217.6 mm, vias 0 -> 1
- net GNDA: track 0.00 -> 195.6 mm, vias 0 -> 6
- net EAD8: track 0.00 -> 174.6 mm, vias 0 -> 8
- net EAD10: track 0.00 -> 158.9 mm, vias 0 -> 4
- net N$59: track 0.00 -> 156.9 mm, vias 0 -> 10
- net N$44: track 0.00 -> 95.9 mm, vias 0 -> 1
- net N$26: track 0.00 -> 87.3 mm
- net N$28: track 0.00 -> 70.5 mm, vias 0 -> 2
- net N$40: track 0.00 -> 37.3 mm, vias 0 -> 3
- net EA7: track 0.00 -> 26.8 mm
- net EA6: track 0.00 -> 26.1 mm
- net EA5: track 0.00 -> 25.4 mm
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- added copper zone on layer 16, net GNDA
- added copper zone on layer 1, net V+
Other:
- board size 181 x 56.6 mm -> 181 x 107.8 mm
- board text added: "BOT"
- board text added: "HBT"
- board text added: "TOP"
