File: Hardware/8ModuleBoard_vr2/8ModuleBoard_vr2.sch (EAGLE design)
At the start: 78 parts, among them CN2 Capsense I/P, Q1 16MHz, T1 BTB16-V, T2 BTB16-V, T3 BTB16-V, T4 BTB16-V, T5 BTB16-V, U1 LM-35, Y1 32.768KHz

Commit message: Updated with Vr2 of Switchboard
Parts:
- removed C10, C11: 0.1uF, SparkFun-Passives:CAP1206
- removed C2: 0.01uF/400V, capacitor-wima:C2.5/2
- removed JP3: USB-Charging, SparkFun-Connectors:USB-A-H
- removed R35: 560R, SparkFun-Resistors:RESISTOR1206
- removed R36: 470R/0.5W, rcl:R-US_0411/3V
- removed R37: 39R/2W, rcl:R-EU_0411/3V
- removed T5: BTB16-V, triac:BT138-V
- removed U$10: RF-LINK_TX, SparkFun-RF:RF-LINK_TX
- removed U1: LM-35, microbuilder:BREAKOUT_SOIC8
- added ANT1: (no value), discrete:ANTENNA
- added D10, D11, D4, D5, D6, D7, D8, D9: (no value), diode:DIODE-SOD123
- added IC2: HT680D, holtek:HT680D
- added JP1: AVR_SPI_PRG_6PTH, SparkFun-Connectors:AVR_SPI_PRG_6PTH
- added K1, K2, K3, K4: JS-M1-9V-4, relay:JS-M1-9V-4
- added LED3: (no value), led:LEDSML1206
- added OK1, OK2, OK3: PC817DIL4, optocoupler:PC817DIL4
- added Q2, Q3, Q4, Q5, Q6: MMBT2222A, SparkFun-DiscreteSemi:TRANSISTOR_NPNMMBT2222A
- added R10, R11, R12, R13: S10K11, varistor:S10K11
- added R14: 10K, SparkFun-Passives:RESISTOR1206
- added R15: 560R, SparkFun-Resistors:RESISTOR1206
- added R16: 33k, SparkFun-Resistors:RESISTOR1206
- added R17, R18, R19, R20: 1K, SparkFun-Resistors:RESISTOR1206
- added S1: SWS008, smd-special:SWS008
- added X1: 22-23-2031, con-molex:22-23-2031
- OK4: value MOC3031M -> MOC3031S; device optocoupler:MOC3031M -> optocoupler:MOC3031S
- OK5, OK6, OK7: value MOC3031M -> MOC3031S; device optocoupler:MOC3031M -> optocoupler:MOC3031S; MF (none) -> FAIRCHILD SEMICONDUCTOR; MPN (none) -> MOC3031SM; OC_FARNELL (none) -> unknown; OC_NEWARK (none) -> 34C1335
- OK8: value MOC3031M -> PC817DIL4; device optocoupler:MOC3031M -> optocoupler:PC817DIL4
- R1: device varistor:S07K11 -> varistor:S10K11
Connections:
- removed net N$17: U1.2
- removed net N$18: U1.3
- removed net N$21: R8.2, U$1.SDA
- removed net N$25: U1.5
- removed net N$26: U1.6
- removed net N$28: U1.7
- removed net N$4 (its old number): OK8.A, R35.2
- removed net N$82: OK8.A2, R36.1
- removed net N$84: OK8.A1, T5.G
- removed net SOCKET: R35.1
- removed net V_TEMP: U1.1
- new net (DIN)TE: IC2.A6, U$2.DATA
- new net (VT)ADOUT: IC2.A9, R14.2
- new net A0: IC2.AD11, S1.16
- new net A1: IC2.AD12, S1.15
- new net A2: IC2.AD14, S1.14
- new net A3: IC2.AD15, S1.13
- new net A4: IC2.DOUT, S1.12
- new net A5: IC2.TE, S1.11
- new net A6: IC2.OSC2, S1.10
- new net A7: IC2.OSC1, S1.9
- new net D10: ATMEGA32U4.PF1(ADC1), IC2.A2
- new net D11: ATMEGA32U4.PF0(ADC0), IC2.A3
- new net D8: ATMEGA32U4.PF5(ADC5), IC2.A0
- new net D9: ATMEGA32U4.PF4(ADC4), IC2.A1
- new net MISO: ATMEGA32U4.PB3(MISO), JP1.3, R20.1
- new net MOSI: ATMEGA32U4.PB2(MOSI), JP1.5, R19.1
- new net N$24: Q2.C, R15.1
- new net N$31: ANT1.1, U$2.ANT
- new net N$32: OK1.EMIT, Q3.B
- new net N$33: D5.A, K11.2, OK1.COL, Q3.C
- new net N$37: D4.C, D5.C
- new net N$38: K12.O
- new net N$41: OK1.A, R17.2
- new net N$43: OK2.EMIT, Q4.B
- new net N$45: D7.A, K21.2, OK2.COL, Q4.C
- new net N$46: D6.C, D7.C
- new net N$47: K22.O
- new net N$50: OK2.A, R18.2
- new net N$51: OK3.EMIT, Q5.B
- new net N$53: D9.A, K31.2, OK3.COL, Q5.C
- new net N$57: D8.C, D9.C
- new net N$58: K32.O
- new net N$65: OK3.A, R19.2
- new net N$66: OK8.EMIT, Q6.B
- new net N$67: D11.A, K41.2, OK8.COL, Q6.C
- new net N$69: D10.C, D11.C
- new net N$73: K42.O
- new net N$77: OK8.A, R20.2
- new net N$8: Q2.B, R14.1
- new net N$83: ATMEGA32U4.PB0(SS), R17.1
- new net OSC1: IC2.A8, R16.1
- new net OSC2: IC2.A7, R16.2
- new net SCK: ATMEGA32U4.PB1(SCK), JP1.4, R18.1
- new net SCL: ATMEGA32U4.PD0(SCL), R7.2, U$1.SCL
- new net SDA: ATMEGA32U4.PD1(SDA), R8.2, U$1.SDA
- net !RESET: now also JP1.1
- net +5V: now also D10.A, D4.A, D6.A, D8.A, IC2.VDD, JP1.2, K11.1, K21.1, K31.1, K41.1, LED3.A, U$2.+5V, X1-1.S; no longer C10.2, C11.1, JP3.VBUS, U1.8
- net DOWN: now also ATMEGA32U4.PB5(ADC12)
- net FAN_ON/OFF: now also ATMEGA32U4.PB6(ADC13)
- net FAN_REG: now also R10.1, R11.1, R12.1, R13.1
- net GND: now also IC2.VSS, JP1.6, OK1.C, OK2.C, OK3.C, Q2.E, Q3.E, Q4.E, Q5.E, Q6.E, S1.1, S1.2, S1.3, S1.4, S1.5, S1.6, S1.7, S1.8, U$2.GND, X1-2.S; no longer C10.1, C11.2, JP3.GND, U1.4
- net LEVEL1: now also ATMEGA32U4.PC6
- net LEVEL2: now also ATMEGA32U4.PC7
- net LEVEL3: now also ATMEGA32U4.PF7(ADC7)
- net LEVEL4: now also ATMEGA32U4.PF6(ADC6)
- net LINE: now also F1.1, K12.P, K22.P, K32.P, K42.P, R10.2, R11.2, R12.2, R13.2; no longer F1.2, R36.2, R37.2, T5.A2
- net LOAD_1: now also K42.S
- net LOAD_2: now also K12.S
- net LOAD_3: now also K22.S
- net N$12: now also Y1.1; no longer Y1.2
- net N$13: now also Y1.2; no longer Y1.1
- net N$20: now also ATMEGA32U4.PE6; no longer R7.2, U$1.SCL
- net N$27: now also LED3.C, R15.2; no longer C2.1, R37.1
- net N$36: now also F1.2; no longer F1.1
- net PLUG_CONTROL: now also K32.S; no longer C2.2, T5.A1
- net RX: now also ATMEGA32U4.PD3(TX)
- net SW-1: now also ATMEGA32U4.PD5
- net SW-2: now also ATMEGA32U4.PD4(ADC8)
- net SW-3: now also ATMEGA32U4.PD6(ADC9)
- net SW-4: now also ATMEGA32U4.PD7(ADC10)
- net TX: now also ATMEGA32U4.PD2(RX)
- net UP: now also ATMEGA32U4.PB4(ADC11)
Other:
- note added: "RF Receiver 434 MHz"
- note added: "RTC Managment"
- note added: "Temperature Sensor Module"
- note added: "Temperature Sensor Removed"
- note removed: "Socket Control"
- moved on the sheet: ATMEGA32U4, B1, C14, C15, C16, C17, C18, C19, C6, C7, C8, C9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

Commit message: Updated with 8 Module Relay Board Design
Parts:
- added 0, 1, 2, 3, 4, 5, 6, 7, 8, 9, DOWN, F_OFF, F_ON, UP: BUTTON-CONDUCTIVESMD, SparkFun-Electromechanical:BUTTON-CONDUCTIVESMD
- added ANT2: (no value), discrete:ANTENNA
- added D12, D13, D14, D15, D16, D17, D18, D19, D20, D21, D22, D23, D24, D25, D26, D27, D28, D29, D30, D31, D32, D33, D34, D35, D36, D37, D38, D39, D40, D41, D42, D43: (no value), diode:DIODE-SOD123
- added IC3: HT680D, holtek:HT680D
- added MASTER: BUTTON-CONDUCTIVE, SparkFun-Electromechanical:BUTTON-CONDUCTIVE
- added R21, R22, R23, R9: 1K, SparkFun-Passives:RESISTOR1206
- added R24: 750K, SparkFun-Passives:RESISTOR1206
- added S2: (no value), SparkFun-Electromechanical:SWITCH-SPDT-SMD-A
- added S3: 219-08J, switch-dil:219-08J
- added TX: RF-LINK_TX, SparkFun-RF:RF-LINK_TX
- added VBAT: (no value), SparkFun-Electromechanical:BATTERY20SMD
Connections:
- new net EA0: IC3.AD11, S3.16
- new net EA1: IC3.AD12, S3.15
- new net EA2: IC3.AD14, S3.14
- new net EA3: IC3.AD15, S3.13
- new net EA4: IC3.DOUT, S3.12
- new net EA5: IC3.TE, S3.11
- new net EA6: IC3.OSC2, S3.10
- new net EA7: IC3.OSC1, S3.9
- new net EAD10: D16.C, D18.C, D20.C, D23.C, D34.C, D36.C, D39.C, D42.C, IC3.A2, R22.1
- new net EAD11: D24.C, D26.C, D28.C, D31.C, D35.C, D37.C, D40.C, D43.C, IC3.A3, R23.1
- new net EAD8: D12.C, D14.C, D17.C, D21.C, D25.C, D29.C, D32.C, D38.C, IC3.A0, R9.1
- new net EAD9: IC3.A1, R21.1
- new net EDOUT: IC3.A9, TX.DATA
- new net EOSC1: IC3.A8, R24.2
- new net EOSC2: IC3.A7, R24.1
- new net GNDA: IC3.A6, IC3.VSS, R21.2, R22.2, R23.2, R9.2, S3.1, S3.2, S3.3, S3.4, S3.5, S3.6, S3.7, S3.8, TX.GND, VBAT.-
- new net N$17: 1.2, D12.A
- new net N$18: 2.2, D13.A
- new net N$26: S2.P, VBAT.+
- new net N$28: S2.S, TX.+5V
- new net N$35: 3.2, D14.A, D15.A
- new net N$40: ANT2.1, TX.ANT
- new net N$42: 4.2, D16.A
- new net N$44: 5.2, D17.A, D18.A
- new net N$48: 6.2, D19.A, D20.A
- new net N$49: 7.2, D21.A, D22.A, D23.A
- new net N$52: 0.2, D27.A, D28.A
- new net N$59: D13.C, D15.C, D19.C, D22.C, D27.C, D30.C, D33.C, D41.C
- new net N$60: D29.A, D30.A, D31.A, UP.2
- new net N$61: 8.2, D24.A
- new net N$68: D36.A, D37.A, F_ON.2
- new net N$74: 9.2, D25.A, D26.A
- new net N$75: D38.A, D39.A, D40.A, DOWN.2
- new net N$76: D32.A, D33.A, D34.A, D35.A, MASTER.2
- new net N$79: D41.A, D42.A, D43.A, F_OFF.2
- new net V+: 0.1, 1.1, 2.1, 3.1, 4.1, 5.1, 6.1, 7.1, 8.1, 9.1, DOWN.1, F_OFF.1, F_ON.1, IC3.VDD, MASTER.1, UP.1
Other:
- note added: "1"
- note added: "10"
- note added: "11"
- note added: "12"
- note added: "13"
- note added: "14"
- note added: "2"
- note added: "3"
- note added: "4"
- note added: "5"
- note added: "6"
- note added: "7"
- note added: "8"
- note added: "9"
- note added: "D0"
- note added: "D1"
- note added: "D2"
- note added: "D3"
- note added: "DOWN"
- note added: "FAN OFF"
- note added: "FAN ON"
- note added: "MASTER"
- note added: "RF Remote Transmitter"
- note added: "UP"
- moved on the sheet: AC-1, AC-2, ANT1, ATMEGA32U4, C1, C18, C19, C3, C4, C5, C6, C7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

Commit message: Updated with 8keyRelayModule firmware files
Other:
- note removed: "LEVEL1"
- note removed: "LEVEL2"
- note removed: "LEVEL3"
- note removed: "LEVEL4"
- note removed: "SOCKET"
Changed lines of the file:
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@@
 <text x="-17.78" y="88.9" size="3.81" layer="104" font="vector" ratio="19">Power Supply Section</text>
 <text x="-96.52" y="-241.3" size="5.08" layer="95" font="vector" ratio="20">Microcontroller Unit</text>
-<text x="33.02" y="-96.52" size="1.778" layer="95">SOCKET</text>
-<text x="33.02" y="-99.06" size="1.778" layer="95">LEVEL4</text>
-<text x="33.02" y="-101.6" size="1.778" layer="95">LEVEL3</text>
-<text x="33.02" y="-104.14" size="1.778" layer="95">LEVEL2</text>
-<text x="33.02" y="-106.68" size="1.778" layer="95">LEVEL1</text>
 <text x="297.18" y="-101.6" size="3.81" layer="95" font="vector" ratio="15">Level-1</text>
 <text x="297.18" y="-142.24" size="3.81" layer="95" font="vector" ratio="15">Level-2</text>
