File: Hardware/8ModuleBoard_vr2/8ModuleBoard_vr2.sch (EAGLE design)
At the start: 163 parts, among them CN2 Capsense I/P, IC2 HT680D, IC3 HT680D, K1 JS-M1-9V-4, K2 JS-M1-9V-4, K3 JS-M1-9V-4, K4 JS-M1-9V-4, Q1 16MHz, Q2 MMBT2222A, Q3 MMBT2222A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

Commit message: Modified 8ModuleBoard_vr2 files
Other:
- note added: "ADD RC SNUBBER CIRCUIT IN FAN REGULATOR"
Changed lines of the file:
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@@
 <wire x1="106.68" y1="-25.4" x2="106.68" y2="134.62" width="6.4516" layer="95"/>
 <text x="322.58" y="-431.8" size="5.08" layer="95" font="vector" ratio="20">RF Remote Transmitter</text>
+<text x="271.78" y="-43.18" size="5.08" layer="95" font="vector" ratio="20">ADD RC SNUBBER CIRCUIT IN FAN REGULATOR</text>
 </plain>
 <instances>
