File: Hardware/Pi_MCU_Backend/pi_mcu_powerBoard.brd (EAGLE design)
At the start: 202.9 x 88 mm, 111 parts, among them CN2 Capsense I/P, IC2 HT680D, K1 RE030012, K2 RE030012, K3 RE030012, K4 RE030012, Q1 IRF540, Q2 MMBT2222A, T1 BTB16-V, T2 BTB16-V, T3 BTB16-V, T4 BTB16-V, T5 BC547, T6 BC547, T7 BC547, T8 BC547, X2 22-23-2031, X4 22-23-2041, X6 22-23-2021, X7 22-23-2021, Y1 32.768KHz

Commit message: modified .brd file
Parts:
- removed D5: 1N4148DO35-7, diode:DO35-7
- removed D6: (no value), diode:D-5
- removed LED3, LED6: (no value), led:LED3MM
- removed Q1: IRF540, transistor-power:TO220BV
- removed R1, R2, R3: (no value), rcl:0207/10
- removed SG1: F/HMB, buzzer:F/HMB
- removed T9: (no value), transistor-neu-to92:TO92-EBC
- removed U$10, U$9: (no value), holes:2,8
- removed X6, X7: 22-23-2021, con-molex:22-23-2021
- added R4, R5, R6, R9: (no value), rcl:0207/10
- added RFLED: (no value), led:LED3MM
- R14: device SparkFun-Passives:1206 -> rcl:0207/10
- moved IC2 16.7 mm to (31.9, 31.4)
- moved R16 15.9 mm to (40.6, 29.0)
- moved R15 11.4 mm to (10.4, 18.6), turned to 90 degrees
- moved C5 8.79 mm to (5.33, 21.2), turned to 0 degrees
- moved Q2 5.35 mm to (17.8, 16.8), turned to 180 degrees
- moved C4 3.06 mm to (64.3, 57.5), turned to 90 degrees
- moved CN2 3.01 mm to (40.2, 5.42), turned to 0 degrees
- moved RN1 2.31 mm to (40.2, 10.9), turned to 0 degrees
- moved R14 1.89 mm to (18.9, 17.3), flipped to the top, turned to 0 degrees
- moved S1 1.73 mm to (17.1, 31.7)
- moved R28 0.97 mm to (111.4, 49.0), flipped to the top, turned to 0 degrees
- moved JP2 0.91 mm to (75.4, 61.1)
- renumbered U$1 to R35, U$11 to R37, U$12 to R38, U$13 to R39, U$14 to R40, U$15 to RTC, U$17 to R41, U$18 to R42, U$19 to R43, U$2 to R36, U$20 to R44, U$21 to RF, U$22 to R45, U$23 to R46, U$24 to R49, U$25 to R51, U$26 to R47, U$27 to R48, U$28 to R50, U$29 to R52
Connections:
- removed net +: Q1.S, R2.2, X6.2
- removed net G: D5.A, LED6.A, SG1.-, T9.E, X6.1, X7.1
- removed net N$45: Q1.G, R2.1, T9.C
- removed net N$46: D6.C, Q1.D, R1.2, X7.2
- removed net N$47: D5.C, R1.1, T9.B
- removed net N$49: D6.A, R3.2, SG1.+
- removed net N$50: LED6.K, R3.1
- net +5V: now also RFLED.A; no longer LED3.A
- net DOWN: now also JP1.35; no longer JP1.23
- net FAN_ON/OFF: now also JP1.37; no longer JP1.21
- net GND: now also R4.1, R5.1, R6.1, R9.1
- net N$27: now also RFLED.K; no longer LED3.K
- net RFD0: now also JP1.15, R4.2; no longer JP1.11
- net RFD1: now also JP1.19, R5.2; no longer JP1.13
- net RFD2: now also JP1.21, R6.2; no longer JP1.15
- net RFD3: now also JP1.23, R9.2; no longer JP1.19
- net SW-1: now also JP1.11; no longer JP1.37
- net SW-2: now also JP1.13; no longer JP1.35
- net SW-3: now also JP1.29; no longer JP1.33
- net UP: now also JP1.33; no longer JP1.29
Routing:
- net G: track 69.7 -> 0.00 mm
- net +: track 59.6 -> 0.00 mm
- net SW-1: track 27.9 -> 65.6 mm, vias 0 -> 2
- net +5V: track 312.7 -> 348.1 mm
- net FAN_ON/OFF: track 55.5 -> 20.5 mm
- net (DIN)TE: track 74.5 -> 45.7 mm
- net SW-2: track 34.4 -> 61.6 mm, vias 0 -> 2
- net (VT)ADOUT: track 43.8 -> 17.5 mm
- net DOWN: track 51.6 -> 27.6 mm
- net GND: track 516.7 -> 497.2 mm, vias 8 -> 6
- net RFD2: track 11.9 -> 31.4 mm
- net RFD1: track 11.4 -> 30.8 mm
- net A2: track 25.4 -> 6.27 mm
- net A1: track 25.9 -> 6.79 mm
- net A3: track 24.9 -> 5.99 mm
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- added copper zone on layer 16, net N$63
- added copper zone on layer 16, net N$72
- removed copper zone on layer 16, net (VT)ADOUT
- removed copper zone on layer 16, net N$42
Other:
- board size 202.9 x 88 mm -> 180.5 x 65 mm
- board text added: "3.3V"
- board text added: "BOT VIEW"
- board text added: "GND"
- board text added: "HBT Vr4"
- board text added: "RX"
- board text added: "TX"
- board text removed: "+5V and GND at RF module short ahe"
- board text removed: "I/P"
- board text removed: "O/P"
