File: Hardware/Pi_MCU_Backend/pi_mcu_powerBoard.sch (EAGLE design)
At the start: 103 parts, among them CN2 Capsense I/P, IC2 HT680D, K1 RE030012, K2 RE030012, K3 RE030012, K4 RE030012, Q1 IRF540, Q2 MMBT2222A, T1 BTB16-V, T2 BTB16-V, T3 BTB16-V, T4 BTB16-V, T5 BC547, T6 BC547, T7 BC547, T8 BC547, X2 22-23-2031, X4 22-23-2041, X6 22-23-2021, X7 22-23-2021, Y1 32.768KHz

Commit message: modified .sch file
Parts:
- removed D5: 1N4148DO35-7, diode:1N4148DO35-7
- removed D6: (no value), diode:DIODE-D-5
- removed LED6: (no value), led:LED3MM
- removed Q1: IRF540, transistor-power:IRF540
- removed R1, R2, R3: (no value), rcl:R-EU_0207/10
- removed SG1: F/HMB, buzzer:F/HMB
- removed T9: (no value), transistor-neu-to92:2N4401-NPN-TO92-EBC
- removed X6, X7: 22-23-2021, con-molex:22-23-2021
- added R4, R5, R6, R9: (no value), rcl:R-EU_0207/10
- C5: device rcl:C-EUC1206 -> rcl:C-USC1206
- R14: device SparkFun-Passives:RESISTOR1206 -> rcl:R-EU_0207/10
- renumbered LED3 to RFLED, U$1 to R35, U$11 to R37, U$12 to R38, U$13 to R39, U$14 to R40, U$15 to RTC, U$17 to R41, U$18 to R42, U$19 to R43, U$2 to R36, U$20 to R44, U$21 to RF, U$22 to R45, U$23 to R46, U$24 to R49, U$25 to R51, U$26 to R47, U$27 to R48, U$28 to R50, U$29 to R52
Connections:
- removed net +: Q1.S, R2.2, X6-2.S
- removed net G: D5.A, LED6.A, SG1.-, T9.E, X6-1.S, X7-1.S
- removed net N$45: Q1.G, R2.1, T9.C
- removed net N$46: D6.C, Q1.D, R1.2, X7-2.S
- removed net N$47: D5.C, R1.1, T9.B
- removed net N$49: D6.A, R3.2, SG1.+
- removed net N$50: LED6.C, R3.1
- net DOWN: now also JP1.GP19; no longer JP1.SCLK
- net FAN_ON/OFF: now also JP1.GP26; no longer JP1.MISO
- net GND: now also R4.1, R5.1, R6.1, R9.1
- net RFD0: now also JP1.GP22, R4.2; no longer JP1.GP17
- net RFD1: now also JP1.MOSI, R5.2; no longer JP1.GP27
- net RFD2: now also JP1.MISO, R6.2; no longer JP1.GP22
- net RFD3: now also JP1.SCLK, R9.2; no longer JP1.MOSI
- net SW-1: now also JP1.GP17; no longer JP1.GP26
- net SW-2: now also JP1.GP27; no longer JP1.GP19
- net SW-3: now also JP1.GP5; no longer JP1.GP13
- net UP: now also JP1.GP13; no longer JP1.GP5
Other:
- note added: "Put Pull Down resistor to RF output pins"
